Commit message: Add files via upload

File: Python Simulation/fetch.urdf (robot description, URDF)
Before this commit: robot fetch_arm, 8 links, 7 joints
Links:
- added link gripper_link, mass 1.5175; collision mesh filename=meshes/gripper_link.STL; visual mesh filename=meshes/gripper_link.dae
- added link l_gripper_finger_link, mass 0.0798; collision box size=0.062 0.013 0.026; visual mesh filename=meshes/l_gripper_finger_link.STL
- added link r_gripper_finger_link, mass 0.0798; collision box size=0.062 0.013 0.026; visual mesh filename=meshes/r_gripper_finger_link.STL
- link elbow_flex_link: geometry collision mesh filename=meshes/elbow_flex_link_collision.STL; visual mesh filename=meshes/elbow_flex_link.dae
- link forearm_roll_link: geometry collision mesh filename=meshes/forearm_roll_link_collision.STL; visual mesh filename=meshes/forearm_roll_link.dae
- link shoulder_lift_link: geometry collision mesh filename=meshes/shoulder_lift_link_collision.STL; visual mesh filename=meshes/shoulder_lift_link.dae
- link shoulder_pan_link: geometry collision mesh filename=meshes/shoulder_pan_link_collision.STL; visual mesh filename=meshes/shoulder_pan_link.dae
- link torso_lift_link: geometry collision mesh filename=meshes/torso_lift_link_collision.STL; visual mesh filename=meshes/torso_lift_link.dae
- link upperarm_roll_link: geometry collision mesh filename=meshes/upperarm_roll_link_collision.STL; visual mesh filename=meshes/upperarm_roll_link.dae
- link wrist_flex_link: geometry collision mesh filename=meshes/wrist_flex_link_collision.STL; visual mesh filename=meshes/wrist_flex_link.dae
- link wrist_roll_link: geometry collision mesh filename=meshes/wrist_roll_link_collision.STL; visual mesh filename=meshes/wrist_roll_link.dae
Joints:
- added joint gripper_axis: type fixed, parent wrist_roll_link, child gripper_link, origin xyz=0.16645 0 0 rpy=0 0 0, axis 0 1 0
- added joint l_gripper_finger_joint: type prismatic, parent gripper_link, child l_gripper_finger_link, origin xyz=0 -0.015425 0 rpy=0 0 0, axis 0 -1 0, limit lower=0.0 upper=0.05 effort=60 velocity=0.05
- added joint r_gripper_finger_joint: type prismatic, parent gripper_link, child r_gripper_finger_link, origin xyz=0 0.015425 0 rpy=0 0 0, axis 0 1 0, limit lower=0.0 upper=0.05 effort=60 velocity=0.05
- joint shoulder_pan_joint: origin xyz=0.119525 0 0.34858 rpy=0 0 0 -> xyz=0.032650 0 0.726010 rpy=0 0 0
